File: pcb/troublemaker/troublemaker.kicad_sch (KiCad schematic)
At the start: 106 parts, among them SW1 sw_eq2, SW10 sw_grain_playback, SW2 sw_eq1, SW3 sw_sub, SW4 sw_bass, SW5 sw_mid, SW6 sw_high, SW7 btn_delay_taptempo, SW8 sw_delay_type, SW9 sw_grain_type, U1 Teensy4.1, U2 CD74HC4067M, U3 CD74HC4067M, U4 CD74HC4067M, U5 CD74HC4067M, U6 CD74HC4067M

Commit message: Added taptempo led, now using SnapEDA teensy and rpi schemes and footprints
Parts:
- removed U1: Teensy4.1, symbol teensy:Teensy4.1
- added IC1: TEENSY_4.1, TEENSY_4.1:TEENSY41, symbol TEENSY_4.1:TEENSY_4.1
- added U1: RASPBERRY_PI_4B_4GB, RASPBERRY_PI_4B_4GB:MODULE_RASPBERRY_PI_4B_4GB, symbol RASPBERRY_PI_4B_4GB:RASPBERRY_PI_4B_4GB
- added taptempo_led: LED, symbol Device:LED
- renumbered Neopixel_bass_gain_reduction to Neopixel_bass_gain_reduction1, Neopixel_bass_out_level to Neopixel_bass_out_level1, Neopixel_high_gain_reduction to Neopixel_high_gain_reduction1, Neopixel_high_out_level to Neopixel_high_out_level1, Neopixel_mid_gain_reduction to Neopixel_mid_gain_reduction1, Neopixel_mid_out_level to Neopixel_mid_out_level1, Neopixel_sub_gain_reduction to Neopixel_sub_gain_reduction1, Neopixel_sub_out_level to Neopixel_sub_out_level1
Connections:
- net rpi_pin19_GPIO10 is gone; now on net neopixel_data: Neopixel_sub_gain_reduction1. (VCC)
- net rpi_pin4_5V is gone; now on net neopixel_data: Neopixel_sub_gain_reduction1. (VCC)
- net 3v3: now also IC1.53 (3.3V_(250_M_A_MAX))
- net GND: now also IC1.69 (GND_4), IC1.70 (GND_5), IC1.71 (GND_6), U1.14 (GND), U1.20 (GND), U1.25 (GND), U1.30 (GND), U1.34 (GND), U1.39 (GND), U1.6 (GND), U1.9 (GND), taptempo_led.1 (K)
- net btn_delay_taptempo: now also IC1.16 (A2)
- net mux1_enable: now also IC1.6 (OUT1D)
- net mux2_enable: now also IC1.7 (RX2)
- net mux3_enable: now also IC1.8 (TX2)
- net mux4_enable: now also IC1.9 (OUT1C)
- net mux5_enable: now also IC1.10 (CS_1)
- net mux_s0: now also IC1.2 (OUT2)
- net mux_s1: now also IC1.3 (LRCLK2)
- net mux_s2: now also IC1.4 (BCLK2)
- net mux_s3: now also IC1.5 (IN2)
- net mux_signal: now also IC1.14 (A0)
- net samlper_5: now also IC1.26 (A12)
- net sampler_1: now also IC1.11 (MOSI)
- net sampler_10: now also IC1.31 (CTX3)
- net sampler_11: now also IC1.32 (OUT1B)
- net sampler_2: now also IC1.12 (MISO)
- net sampler_3: now also IC1.24 (A10)
- net sampler_4: now also IC1.25 (A11)
- net sampler_6: now also IC1.27 (A13)
- net sampler_7: now also IC1.28 (RX7)
- net sampler_8: now also IC1.29 (TX7)
- net sampler_9: now also IC1.30 (CRX3)
- net sampler_stop: now also IC1.23 (A9)
- net sw_bass: now also IC1.19 (A5)
- net sw_delay_type: now also IC1.15 (A1)
- net sw_eq1: now also IC1.22 (A8)
- net sw_eq2: now also IC1.21 (A7)
- net sw_grain_playback: now also IC1.39 (A15)
- net sw_grain_type: now also IC1.38 (A14)
- net sw_high: now also IC1.17 (A3)
- net sw_mid: now also IC1.18 (A4)
- net sw_sub: now also IC1.20 (A6)
- net at Neopixel_high_gain_reduction1. (VCC): now also Neopixel_mid_out_level1. (VCC); no longer Neopixel_high_out_level1. (VCC)
- net at Neopixel_high_out_level1. (VCC): no longer Neopixel_high_gain_reduction1. (VCC)
- net at Neopixel_mid_out_level1. (VCC): now also Neopixel_mid_gain_reduction1. (VCC); no longer Neopixel_high_gain_reduction1. (VCC)
- net at Neopixel_bass_out_level1. (VCC): now also Neopixel_bass_gain_reduction1. (VCC); no longer Neopixel_mid_gain_reduction1. (VCC)
- net at Neopixel_bass_gain_reduction1. (VCC): now also Neopixel_sub_out_level1. (VCC); no longer Neopixel_bass_out_level1. (VCC)
- net neopixel_data: now reaches Neopixel_sub_gain_reduction1. (VCC)
- net neopixel_data: now also U1.19 (GPIO10/SPI_MOSI); no longer Neopixel_sub_out_level1. (VCC)
- new net: Neopixel_high_gain_reduction1. (VCC), Neopixel_high_out_level1. (VCC) (x4)
- new net: Neopixel_high_gain_reduction1. (VCC), Neopixel_mid_out_level1. (VCC) (x3)
- new net: U1.1 (3V3), U1.17 (3V3)
- new net: U1.S1 (SHIELD), U1.S2 (SHIELD), U1.S3 (SHIELD), U1.S4 (SHIELD)
- new net: Neopixel_bass_out_level1. (VCC), Neopixel_mid_gain_reduction1. (VCC) (x4)
- new net: Neopixel_mid_gain_reduction1. (VCC), Neopixel_mid_out_level1. (VCC) (x3)
- new net: Neopixel_bass_gain_reduction1. (VCC), Neopixel_bass_out_level1. (VCC) (x3)
- new net: Neopixel_sub_gain_reduction1. (VCC), Neopixel_sub_out_level1. (VCC) (x4)
- new net: Neopixel_bass_gain_reduction1. (VCC), Neopixel_sub_out_level1. (VCC) (x3)
- new net +5V: Neopixel_sub_gain_reduction1. (VCC), U1.2 (5V), U1.4 (5V)
- new net taptempo_LED: U1.16 (GPIO23/GPIO_GEN4), taptempo_led.2 (A)
- now unconnected: Neopixel_high_out_level1. (VCC), Neopixel_high_out_level1. (VCC)
Other:
- note added: "0.2"
- note added: "Skipped because of onboard LED"
- note removed: "0.1"
- moved on the sheet: SW7

Commit message: Added missing stuff on schematic, PCB layout WIP
Parts:
- added J1: neopixel_data_RPI19_GPIO10, Connector_PinHeader_1.00mm:PinHeader_1x01_P1.00mm_Vertical, symbol Connector_Generic:Conn_01x01
- added J3: 5V_RPI2_OR_4, Connector_PinHeader_1.00mm:PinHeader_1x01_P1.00mm_Vertical, symbol Connector_Generic:Conn_01x01
- added J4: GND_RPI34, Connector_PinHeader_1.00mm:PinHeader_1x01_P1.00mm_Vertical, symbol Connector_Generic:Conn_01x01
- added J5: Conn_01x12, Connector_PinHeader_2.00mm:PinHeader_1x12_P2.00mm_Vertical, symbol Connector_Generic:Conn_01x12
- added RV39: pot_dly_lfo_depth, Potentiometer_THT:Potentiometer_Alps_RK09K_Single_Vertical, symbol Device:R_Potentiometer
- added SW11: btn_sampler_stop, leozorLib:arcade_service_button_leozor, symbol Switch:SW_Push
- C1, C2, C3, C4, C5: footprint (none) -> Capacitor_THT:CP_Radial_D5.0mm_P2.00mm
- Neopixel_bass_gain_reduction1, Neopixel_bass_out_level1, Neopixel_high_gain_reduction1, Neopixel_high_out_level1, Neopixel_mid_gain_reduction1, Neopixel_mid_out_level1, Neopixel_sub_gain_reduction1, Neopixel_sub_out_level1: footprint (none) -> leozorLib:Neopixel-8LED
- RV1, RV10, RV11, RV12, RV13, RV14, RV15, RV16, RV17, RV18, RV19, RV2, RV20, RV21, RV22, RV23, RV24, RV25, RV26, RV27, RV28, RV29, RV3, RV30, RV31, RV32, RV33, RV34, RV35, RV36, RV37, RV38, RV4, RV47, RV48, RV49, RV5, RV50, RV51, RV52, RV53, RV54, RV55, RV56, RV57, RV58, RV59, RV6, RV60, RV61, RV62, RV63, RV64, RV65, RV66, RV67, RV68, RV69, RV7, RV70, RV71, RV72, RV73, RV74, RV75, RV76, RV77, RV78, RV79, RV8, RV80, RV81, RV82, RV83, RV84, RV85, RV9: footprint (none) -> Potentiometer_THT:Potentiometer_Alps_RK09K_Single_Vertical
- SW1, SW10, SW2, SW3, SW4, SW5, SW6, SW8, SW9: footprint (none) -> leozorLib:SW_SPDT_red_leozor
- SW7: footprint (none) -> leozorLib:arcade_service_button_leozor
- U2, U3, U4, U5, U6: footprint Package_SO:SOIC-24W_7.5x15.4mm_P1.27mm -> leozorLib:Breakout_HC4067_PTH_Only
- taptempo_led1: renamed from taptempo_led; footprint (none) -> LED_THT:LED_D3.0mm
Connections:
- net +5V: now also Neopixel_sub_gain_reduction1.7 (VCC), J3.1 (Pin_1); no longer Neopixel_sub_gain_reduction1. (VCC)
- net 3v3: now also RV39.1
- net GND: now also Neopixel_sub_gain_reduction1.5 (GND), Neopixel_sub_gain_reduction1.8 (GND), J4.1 (Pin_1), J5.12 (Pin_12), RV39.3, SW11.1; no longer Neopixel_sub_gain_reduction1. (VCC)
- net neopixel_data: now also Neopixel_sub_gain_reduction1.6 (DATA_IN), J1.1 (Pin_1); no longer Neopixel_sub_gain_reduction1. (VCC), U1.19 (GPIO10/SPI_MOSI)
- net samlper_5: now also J5.5 (Pin_5)
- net sampler_1: now also J5.1 (Pin_1)
- net sampler_10: now also J5.10 (Pin_10)
- net sampler_11: now also J5.11 (Pin_11)
- net sampler_2: now also J5.2 (Pin_2)
- net sampler_3: now also J5.3 (Pin_3)
- net sampler_4: now also J5.4 (Pin_4)
- net sampler_6: now also J5.6 (Pin_6)
- net sampler_7: now also J5.7 (Pin_7)
- net sampler_8: now also J5.8 (Pin_8)
- net sampler_9: now also J5.9 (Pin_9)
- net sampler_stop: now also SW11.2
- net at RV59.2: now also U5.6 (I3); no longer U5.7 (I2)
- net at RV72.2: now also U6.9 (I0); no longer U5.16 (I15)
- net at RV77.2: now also U6.4 (I5); no longer U6.5 (I4)
- net at RV62.2: now also U5.3 (I6); no longer U5.4 (I5)
- net at RV71.2: now also U5.16 (I15); no longer U5.17 (I14)
- net at RV70.2: now also U5.17 (I14); no longer U5.18 (I13)
- net at RV69.2: now also U5.18 (I13); no longer U5.19 (I12)
- net at U5.2 (I7): now also RV63.2; no longer RV64.2
- net at RV68.2: now also U5.19 (I12); no longer U5.20 (I11)
- net at RV67.2: now also U5.20 (I11); no longer U5.21 (I10)
- net at RV66.2: now also U5.21 (I10); no longer U5.22 (I9)
- net at RV65.2: now also U5.22 (I9); no longer U5.23 (I8)
- net at RV61.2: now also U5.4 (I5); no longer U5.5 (I4)
- net at RV60.2: now also U5.5 (I4); no longer U5.6 (I3)
- net at RV58.2: now also U5.7 (I2); no longer U5.8 (I1)
- net at RV57.2: now also U5.8 (I1); no longer U5.9 (I0)
- net at RV73.2: now also U6.8 (I1); no longer U6.9 (I0)
- net at RV51.2: now also U4.20 (I11); no longer U4.21 (I10)
- net at RV55.2: now also U4.16 (I15); no longer U4.17 (I14)
- net at RV56.2: now also U5.9 (I0); no longer U4.16 (I15)
- net at RV54.2: now also U4.17 (I14); no longer U4.18 (I13)
- net at RV84.2: now also U6.19 (I12); no longer U6.20 (I11)
- net at RV49.2: now also U4.22 (I9); no longer U4.23 (I8)
- net at RV52.2: now also U4.19 (I12); no longer U4.20 (I11)
- net at RV82.2: now also U6.21 (I10); no longer U6.22 (I9)
- net at U4.2 (I7): now also RV39.2; no longer RV48.2
- net at RV80.2: now also U6.23 (I8); no longer U6.2 (I7)
- net at U6.18 (I13): now also RV85.2
- net at RV83.2: now also U6.20 (I11); no longer U6.21 (I10)
- net at RV81.2: now also U6.22 (I9); no longer U6.23 (I8)
- net at RV79.2: now also U6.2 (I7); no longer U6.3 (I6)
- net at RV78.2: now also U6.3 (I6); no longer U6.4 (I5)
- net at RV76.2: now also U6.5 (I4); no longer U6.6 (I3)
- net at RV75.2: now also U6.6 (I3); no longer U6.7 (I2)
- net at RV74.2: now also U6.7 (I2); no longer U6.8 (I1)
- net at RV50.2: now also U4.21 (I10); no longer U4.22 (I9)
- net at RV53.2: now also U4.18 (I13); no longer U4.19 (I12)
- new net: Neopixel_high_gain_reduction1.1 (GND), Neopixel_high_out_level1.5 (GND)
- new net: Neopixel_high_gain_reduction1.2 (DATA_OUT), Neopixel_high_out_level1.6 (DATA_IN)
- new net: Neopixel_high_gain_reduction1.3 (VCC), Neopixel_high_out_level1.7 (VCC)
- new net: Neopixel_high_gain_reduction1.4 (GND), Neopixel_high_out_level1.8 (GND)
- new net: Neopixel_high_gain_reduction1.5 (GND), Neopixel_mid_out_level1.1 (GND)
- new net: Neopixel_high_gain_reduction1.6 (DATA_IN), Neopixel_mid_out_level1.2 (DATA_OUT)
- new net: Neopixel_high_gain_reduction1.7 (VCC), Neopixel_mid_out_level1.3 (VCC)
- new net: Neopixel_high_gain_reduction1.8 (GND), Neopixel_mid_out_level1.4 (GND)
- new net: RV64.2, U5.23 (I8)
- new net: Neopixel_mid_gain_reduction1.1 (GND), Neopixel_mid_out_level1.5 (GND)
- new net: Neopixel_mid_gain_reduction1.2 (DATA_OUT), Neopixel_mid_out_level1.6 (DATA_IN)
- new net: Neopixel_mid_gain_reduction1.3 (VCC), Neopixel_mid_out_level1.7 (VCC)
- new net: Neopixel_mid_gain_reduction1.4 (GND), Neopixel_mid_out_level1.8 (GND)
- new net: Neopixel_bass_out_level1.1 (GND), Neopixel_mid_gain_reduction1.5 (GND)
- new net: Neopixel_bass_out_level1.2 (DATA_OUT), Neopixel_mid_gain_reduction1.6 (DATA_IN)
- new net: Neopixel_bass_out_level1.3 (VCC), Neopixel_mid_gain_reduction1.7 (VCC)
- new net: Neopixel_bass_out_level1.4 (GND), Neopixel_mid_gain_reduction1.8 (GND)
- new net: RV48.2, U4.23 (I8)
- new net: Neopixel_bass_gain_reduction1.1 (GND), Neopixel_bass_out_level1.5 (GND)
- new net: Neopixel_bass_gain_reduction1.2 (DATA_OUT), Neopixel_bass_out_level1.6 (DATA_IN)
- new net: Neopixel_bass_gain_reduction1.3 (VCC), Neopixel_bass_out_level1.7 (VCC)
- new net: Neopixel_bass_gain_reduction1.4 (GND), Neopixel_bass_out_level1.8 (GND)
- new net: Neopixel_sub_gain_reduction1.1 (GND), Neopixel_sub_out_level1.5 (GND)
- new net: Neopixel_sub_gain_reduction1.2 (DATA_OUT), Neopixel_sub_out_level1.6 (DATA_IN)
- new net: Neopixel_sub_gain_reduction1.3 (VCC), Neopixel_sub_out_level1.7 (VCC)
- new net: Neopixel_sub_gain_reduction1.4 (GND), Neopixel_sub_out_level1.8 (GND)
- new net: Neopixel_bass_gain_reduction1.5 (GND), Neopixel_sub_out_level1.1 (GND)
- new net: Neopixel_bass_gain_reduction1.6 (DATA_IN), Neopixel_sub_out_level1.2 (DATA_OUT)
- new net: Neopixel_bass_gain_reduction1.7 (VCC), Neopixel_sub_out_level1.3 (VCC)
- new net: Neopixel_bass_gain_reduction1.8 (GND), Neopixel_sub_out_level1.4 (GND)
Other:
- moved on the sheet: RV47, RV48, RV49, RV50, RV51, RV52, RV53, RV54, RV55, RV56, RV57

Commit message: JLCPCB DRC, pots are connected to muxers, rearranged scheme, added missing LED resistor and pin header
Parts:
- added J2: taptempo_led_RPI16_GPIO23, Connector_PinHeader_1.00mm:PinHeader_1x01_P1.00mm_Vertical, symbol Connector_Generic:Conn_01x01
- added R1: R 75ohm, Resistor_THT:R_Axial_DIN0207_L6.3mm_D2.5mm_P10.16mm_Horizontal, symbol Device:R
- taptempo_led1: value LED -> LED chartreuse 1.8-2V, 20mA
Connections:
- net 3v3: no longer U3.22 (I9), U3.23 (I8)
- net taptempo_LED: now also J2.1 (Pin_1), R1.1; no longer U1.16 (GPIO23/GPIO_GEN4), taptempo_led1.2 (A)
- net at RV59.2: now also U4.23 (I8); no longer U5.6 (I3)
- net at RV28.2: now also U3.9 (I0); no longer U3.20 (I11)
- net at RV72.2: now also U6.7 (I2); no longer U6.9 (I0)
- net at RV77.2: now also U6.2 (I7); no longer U6.4 (I5)
- net at RV25.2: now also U2.18 (I13)
- net at RV39.2: now also U3.19 (I12); no longer U4.2 (I7)
- net at RV31.2: now also U3.6 (I3); no longer U3.17 (I14)
- net at RV38.2: now also U3.21 (I10); no longer U4.4 (I5)
- net at U3.16 (I15): now also RV50.2; no longer RV32.2
- net at U3.18 (I13): now also RV48.2; no longer RV30.2
- net at RV29.2: now also U3.8 (I1); no longer U3.19 (I12)
- net at U3.2 (I7): now also RV35.2; no longer RV24.2
- net at RV27.2: now also U2.16 (I15); no longer U3.21 (I10)
- net at U3.3 (I6): now also RV34.2; no longer RV23.2
- net at U3.4 (I5): now also RV33.2; no longer RV22.2
- net at U3.5 (I4): now also RV32.2; no longer RV21.2
- net at RV20.2: now also U5.4 (I5); no longer U3.6 (I3)
- net at U3.7 (I2): now also RV30.2; no longer RV19.2
- net at RV18.2: now also U5.8 (I1); no longer U3.8 (I1)
- net at RV17.2: now also U5.21 (I10); no longer U3.9 (I0)
- net at RV62.2: now also U4.20 (I11); no longer U5.3 (I6)
- net at U5.16 (I15): no longer RV71.2
- net at U5.17 (I14): no longer RV70.2
- net at U5.2 (I7): now also RV21.2; no longer RV63.2
- net at RV66.2: now also U4.16 (I15); no longer U5.21 (I10)
- net at U5.22 (I9): now also RV22.2; no longer RV65.2
- net at U5.23 (I8): now also RV16.2; no longer RV64.2
- net at RV61.2: now also U4.21 (I10); no longer U5.4 (I5)
- net at U5.5 (I4): now also RV14.2; no longer RV60.2
- net at U5.7 (I2): now also RV13.2; no longer RV58.2
- net at RV57.2: now also U4.3 (I6); no longer U5.8 (I1)
- net at U5.9 (I0): now also RV12.2; no longer RV56.2
- net at U2.19 (I12): now also RV24.2; no longer RV13.2
- net at U4.7 (I2): now also RV53.2; no longer RV35.2
- net at U2.20 (I11): now also RV23.2; no longer RV12.2
- net at RV73.2: now also U6.6 (I3); no longer U6.8 (I1)
- net at RV51.2: now also U4.9 (I0); no longer U4.20 (I11)
- net at RV37.2: now also U3.22 (I9); no longer U4.5 (I4)
- net at RV55.2: now also U4.5 (I4); no longer U4.16 (I15)
- net at RV54.2: now also U4.6 (I3); no longer U4.17 (I14)
- net at RV47.2: now also U3.20 (I11); no longer U4.3 (I6)
- net at RV84.2: now also U6.17 (I14); no longer U6.19 (I12)
- net at RV49.2: now also U3.17 (I14); no longer U4.22 (I9)
- net at U4.19 (I12): now also RV63.2; no longer RV52.2
- net at RV82.2: now also U6.19 (I12); no longer U6.21 (I10)
- net at RV80.2: now also U6.21 (I10); no longer U6.23 (I8)
- net at U6.16 (I15): now also RV85.2
- net at U6.18 (I13): now also RV83.2; no longer RV85.2
- net at RV79.2: now also U6.22 (I9); no longer U6.2 (I7)
- net at U6.20 (I11): now also RV81.2; no longer RV83.2
- net at RV78.2: now also U6.23 (I8); no longer U6.3 (I6)
- net at RV76.2: now also U6.3 (I6); no longer U6.5 (I4)
- net at RV75.2: now also U6.4 (I5); no longer U6.6 (I3)
- net at RV74.2: now also U6.5 (I4); no longer U6.7 (I2)
- net at RV15.2: now also U5.3 (I6); no longer U2.17 (I14)
- net at RV26.2: now also U2.17 (I14)
- net at RV36.2: now also U3.23 (I8); no longer U4.6 (I3)
- net at U4.8 (I1): now also RV52.2; no longer RV34.2
- net at U4.18 (I13): now also RV64.2; no longer RV53.2
- new net: R1.2, taptempo_led1.2 (A)
- new net: RV19.2, U5.6 (I3)
- new net: RV58.2, U4.2 (I7)
- new net: RV56.2, U4.4 (I5)
- new net: RV70.2, U6.9 (I0)
- new net: RV60.2, U4.22 (I9)
- new net: RV71.2, U6.8 (I1)
- new net: RV65.2, U4.17 (I14)
Other:
- moved on the sheet: C1, C2, C3, C4, C5, IC1, J1, J3, J4, J5, Neopixel_bass_gain_reduction1, Neopixel_bass_out_level1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

Commit message: Added symbols and footprints
Parts:
- C1, C2, C3, C4, C5: symbol Device:C_Small -> Library:C_Small
- IC1: symbol TEENSY_4.1:TEENSY_4.1 -> Library:TEENSY_4.1
- J1, J2, J3, J4: symbol Connector_Generic:Conn_01x01 -> Library:Conn_01x01
- J5: symbol Connector_Generic:Conn_01x12 -> Library:Conn_01x12
- Neopixel_bass_gain_reduction1, Neopixel_bass_out_level1, Neopixel_high_gain_reduction1, Neopixel_high_out_level1, Neopixel_mid_gain_reduction1, Neopixel_mid_out_level1, Neopixel_sub_gain_reduction1, Neopixel_sub_out_level1: symbol leozorLib:Neopixel-8LED -> Library:Neopixel-8LED
- R1: symbol Device:R -> Library:R
- RV1, RV10, RV11, RV12, RV13, RV14, RV15, RV16, RV17, RV18, RV19, RV2, RV20, RV21, RV22, RV23, RV24, RV25, RV26, RV27, RV28, RV29, RV3, RV30, RV31, RV32, RV33, RV34, RV35, RV36, RV37, RV38, RV39, RV4, RV47, RV48, RV49, RV5, RV50, RV51, RV52, RV53, RV54, RV55, RV56, RV57, RV58, RV59, RV6, RV60, RV61, RV62, RV63, RV64, RV65, RV66, RV67, RV68, RV69, RV7, RV70, RV71, RV72, RV73, RV74, RV75, RV76, RV77, RV78, RV79, RV8, RV80, RV81, RV82, RV83, RV84, RV85, RV9: symbol Device:R_Potentiometer -> Library:R_Potentiometer
- SW1, SW10, SW2, SW3, SW4, SW5, SW6, SW8, SW9: symbol Switch:SW_SPDT -> Library:SW_SPDT
- SW11, SW7: symbol Switch:SW_Push -> Library:SW_Push
- U1: symbol RASPBERRY_PI_4B_4GB:RASPBERRY_PI_4B_4GB -> Library:RASPBERRY_PI_4B_4GB
- U2, U3, U4, U5, U6: symbol 74xx:CD74HC4067M -> Library:CD74HC4067M
- taptempo_led1: symbol Device:LED -> Library:LED
